File: test8.kicad_sch (KiCad schematic)
At the start: 21 parts, among them J1 Conn_01x10_Socket, J2 Conn_01x10_Socket, J3 Conn_01x02_Pin, J4 Conn_01x03_Pin, J5 Conn_01x03_Pin, J6 Conn_01x03_Pin, J7 Conn_01x10_Socket, J8 Conn_01x10_Socket, U1 74HC165, U2 74HC165, U3 AMS1117-3.3, U4 ESP32-WROOM-32, U5 74HC595, U6 74HC595

Commit message: исправлены разъемы 2мм на 2,54
Parts:
- J1, J2, J7, J8: footprint main:PinHeader_2x05_P2.00mm_Vertical -> main:PinHeader_2x05_P2.54mm_Vertical
- J4, J5, J6: footprint main:PinSocket_1x03_P2.00mm_Vertical -> main:PinHeader_1x03_P2.54mm_Vertical
Changed lines of the file:
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@@
 			)
 		)
-		(property "Footprint" "main:PinHeader_2x05_P2.00mm_Vertical"
+		(property "Footprint" "main:PinHeader_2x05_P2.54mm_Vertical"
 			(at 231.14 80.01 0)
 			(effects
@@
 			)
 		)
-		(property "Footprint" "main:PinHeader_2x05_P2.00mm_Vertical"
+		(property "Footprint" "main:PinHeader_2x05_P2.54mm_Vertical"
 			(at 43.18 73.66 0)
 			(effects
@@
 			)
 		)
-		(property "Footprint" "main:PinSocket_1x03_P2.00mm_Vertical"
+		(property "Footprint" "main:PinHeader_1x03_P2.54mm_Vertical"
 			(at 204.47 40.64 0)
 			(effects
@@
 			)
 		)
-		(property "Footprint" "main:PinHeader_2x05_P2.00mm_Vertical"
+		(property "Footprint" "main:PinHeader_2x05_P2.54mm_Vertical"
 			(at 43.18 128.27 0)
 			(effects
@@
 			)
 		)
-		(property "Footprint" "main:PinSocket_1x03_P2.00mm_Vertical"
+		(property "Footprint" "main:PinHeader_1x03_P2.54mm_Vertical"
 			(at 168.91 55.88 0)
 			(effects
@@
 			)
 		)
-		(property "Footprint" "main:PinHeader_2x05_P2.00mm_Vertical"
+		(property "Footprint" "main:PinHeader_2x05_P2.54mm_Vertical"
 			(at 231.14 120.65 0)
 			(effects
@@
 			)
 		)
-		(property "Footprint" "main:PinSocket_1x03_P2.00mm_Vertical"
+		(property "Footprint" "main:PinHeader_1x03_P2.54mm_Vertical"
 			(at 187.96 40.64 0)
 			(effects
